File: ECE411 Capstone/ECE411 Capstone.kicad_pcb (KiCad board)
At the start: 2 copper layers, 1 part

Commit message: Updated PCB Layout + Routes
Parts:
- removed REF**: Arduino_Nano, Module:Arduino_Nano
- added C1: 0.1uF, Capacitor_SMD:C_01005_0402Metric, B.Cu at (144.0, 92.5)
- added C2: 0.1uF, Capacitor_SMD:C_01005_0402Metric, B.Cu at (135.4, 114.6)
- added C3: 0.1uF, Capacitor_SMD:C_01005_0402Metric, B.Cu at (173.5, 114.6)
- added C4: 0.1uF, Capacitor_SMD:C_01005_0402Metric, B.Cu at (154.4, 114.6)
- added C5: 0.1uF, Capacitor_SMD:C_01005_0402Metric, B.Cu at (163.1, 92.5)
- added C6: 0.1uF, Capacitor_SMD:C_01005_0402Metric, B.Cu at (182.1, 92.5)
- added D1: DIODE, Diode_SMD:D_SOD-123, F.Cu at (144.8, 75.2)
- added D10: WS2812B, LED_SMD:LED_WS2812B_PLCC4_5.0x5.0mm_P3.2mm, B.Cu at (158.8, 94.0)
- added D11: WS2812B, LED_SMD:LED_WS2812B_PLCC4_5.0x5.0mm_P3.2mm, B.Cu at (177.8, 113.0)
- added D12: WS2812B, LED_SMD:LED_WS2812B_PLCC4_5.0x5.0mm_P3.2mm, B.Cu at (139.7, 113.0)
- added D2: DIODE, Diode_SMD:D_SOD-123, F.Cu at (148.1, 75.2)
- added D3: DIODE, Diode_SMD:D_SOD-123, F.Cu at (163.8, 75.2)
- added D4: DIODE, Diode_SMD:D_SOD-123, F.Cu at (167.1, 75.2)
- added D5: DIODE, Diode_SMD:D_SOD-123, F.Cu at (182.9, 75.2)
- added D6: DIODE, Diode_SMD:D_SOD-123, F.Cu at (186.2, 75.2)
- added D7: WS2812B, LED_SMD:LED_WS2812B_PLCC4_5.0x5.0mm_P3.2mm, B.Cu at (139.7, 94.0)
- added D8: WS2812B, LED_SMD:LED_WS2812B_PLCC4_5.0x5.0mm_P3.2mm, B.Cu at (177.8, 94.0)
- added D9: WS2812B, LED_SMD:LED_WS2812B_PLCC4_5.0x5.0mm_P3.2mm, B.Cu at (158.8, 113.0)
- added OL1: OLED, KBD Keyboard stuff:OLED_v2, F.Cu at (141.0, 66.5)
- added R1: 4.7k, Resistor_SMD:R_0201_0603Metric, B.Cu at (122.4, 96.0)
- added SW1: RST Pin, Button_Switch_SMD:SW_Push_1P1T_NO_6x6mm_H9.5mm, B.Cu at (118.4, 100.3)
- added SW2: SW_Push, Mechanical switches:MXOnly-1U-NoLED, F.Cu at (139.7, 87.4)
- added SW3: SW_Push, Mechanical switches:MXOnly-1U-NoLED, F.Cu at (139.7, 106.4)
- added SW4: SW_Push, Mechanical switches:MXOnly-1U-NoLED, F.Cu at (158.8, 87.4)
- added SW5: SW_Push, Mechanical switches:MXOnly-1U-NoLED, F.Cu at (158.8, 106.4)
- added SW6: SW_Push, Mechanical switches:MXOnly-1U-NoLED, F.Cu at (177.8, 87.4)
- added SW7: SW_Push, Mechanical switches:MXOnly-1U-NoLED, F.Cu at (177.8, 106.4)
- added U1: Sparkfun_Pro_Micro, KBD Keyboard stuff:ProMicro_v3, F.Cu at (118.9, 78.4)
Routing:
- net VCC: track 0.00 -> 220.7 mm
- net GND: track 0.00 -> 211.4 mm
- net Column_C: track 0.00 -> 93.1 mm
- net Column_B: track 0.00 -> 75.2 mm
- net Row_B: track 0.00 -> 63.5 mm
- net Row_A: track 0.00 -> 61.2 mm
- net Column_A: track 0.00 -> 50.3 mm
- net SCL: track 0.00 -> 40.1 mm
- net SDA: track 0.00 -> 36.4 mm
- net RST: track 0.00 -> 32.6 mm
- net Net-(D4-Pad1): track 0.00 -> 26.9 mm
- net Net-(D6-Pad1): track 0.00 -> 26.9 mm
- net Net-(D2-Pad1): track 0.00 -> 26.9 mm
- net Net-(D11-Pad4): track 0.00 -> 24.1 mm
- net Net-(D12-Pad4): track 0.00 -> 15.5 mm
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- added copper zone on B.Cu, net GND
- added copper zone on F.Cu, net VCC

Commit message: Updated Schematic + PCB for review
Parts:
- moved C1 0.76 mm to (144.0, 93.2)
- moved C2 0.76 mm to (135.4, 115.3)
- moved C3 0.76 mm to (173.5, 115.3)
- moved C4 0.76 mm to (154.4, 115.3)
- moved C5 0.76 mm to (163.1, 93.2)
- moved C6 0.76 mm to (182.1, 93.2)
- moved D10 0.76 mm to (158.8, 94.7)
- moved D11 0.76 mm to (177.8, 113.8)
- moved D12 0.76 mm to (139.7, 113.8)
- moved D7 0.76 mm to (139.7, 94.7)
- moved D8 0.76 mm to (177.8, 94.7)
- moved D9 0.76 mm to (158.8, 113.8)
- moved SW2 0.76 mm to (139.7, 88.1)
- moved SW3 0.76 mm to (139.7, 107.2)
- moved SW4 0.76 mm to (158.8, 88.1)
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Connections:
- U1 pad 19: Row_B -> Row_A
- U1 pad 20: Row_A -> Row_B
Routing:
- net GND: track 211.4 -> 274.4 mm
- net Column_A: track 50.3 -> 31.2 mm
- net VCC: track 220.7 -> 217.3 mm
- net Column_C: track 93.1 -> 90.4 mm
- net Column_B: track 75.2 -> 73.1 mm
- net Row_A: track 61.2 -> 60.5 mm
- net Net-(D6-Pad1): track 26.9 -> 27.4 mm
- net Net-(D5-Pad1): track 6.51 -> 7.02 mm
- net Net-(D4-Pad1): track 26.9 -> 27.4 mm
- net Net-(D3-Pad1): track 6.51 -> 7.02 mm
- net Net-(D2-Pad1): track 26.9 -> 27.4 mm
- net Net-(D1-Pad1): track 6.51 -> 7.02 mm
- net Net-(D11-Pad4): track 24.1 -> 23.6 mm
Other:
- board text added: "ECE 411 Team 1 David Dinh David Brown Danny Tran Jonathan Cruz"
- board text added: "U1"

Commit message: Final CAD layout
Parts:
- C1, C2, C3, C4, C5, C6: footprint Capacitor_SMD:C_01005_0402Metric -> Capacitor_SMD:C_0805_2012Metric
- moved C2 0.71 mm to (135.1, 114.7)
- moved C6 0.69 mm to (182.4, 93.9)
- moved C3 0.69 mm to (173.2, 114.7)
- moved C4 0.69 mm to (154.2, 114.7)
- moved C5 0.69 mm to (163.3, 93.9)
- moved C1 0.67 mm to (144.3, 93.9)
- moved R1 0.51 mm to (122.4, 96.5)
Routing:
- net GND: track 274.4 -> 34.7 mm, vias 0 -> 18
- net RST: track 32.6 -> 39.5 mm
- net VCC: track 217.3 -> 214.4 mm
- net Column_B: track 73.1 -> 75.6 mm
- net Column_C: track 90.4 -> 92.8 mm
- net Row_B: track 63.2 -> 62.5 mm
- added copper zone on F.Cu, net GND
- removed copper zone on F.Cu, net VCC
Other:
- board outline added: 83.1 x 62.7 mm
- board text added: "ECE 411 Team 1 Version 1.0 11/17/2022"
- board text removed: "ECE 411 Team 1 David Dinh David Brown Danny Tran Jonathan Cruz"
